Commit message: 更新README 增加empty_world_paper

File: model/xacro/omni3robot/omni3robot.xacro (robot description, xacro)
@@ -6,8 +6,12 @@
   <xacro:arg name="pkg_path" default=""/>
   <xacro:include filename="description.gazebo"/>
+  <xacro:include filename="controller.gazebo"/>
+  <xacro:property name="base_mass" value="0.2203"/>
+  <xacro:property name="hub_mass" value="0.0579"/>
+  <xacro:property name="roller_mass" value="0.0023"/>
   <link name="base_link">
     <inertial>
       <origin xyz="-2.60873786585806E-05 0.000243250065461549 0.00991609422071794" rpy="0 0 0" />
-      <mass value="0.220390933719744" />
+      <mass value="${base_mass}" />
       <inertia
       ixx="9.60338008936991E-05" ixy="6.90711247235453E-08" ixz="2.92326723956294E-08"
@@ -31,5 +35,5 @@
     <inertial>
       <origin xyz="2.56280149801462E-05 8.27907396198074E-05 6.93889390390723E-18" rpy="0 0 0" />
-      <mass value="0.0479080577376475" />
+      <mass value="${hub_mass}" />
       <inertia
       ixx="6.84765795190242E-06" ixy="2.68210543382495E-08" ixz="-1.90755783989393E-09"
@@ -59,5 +63,5 @@
     <inertial>
       <origin xyz="0 -2.08166817117217E-17 8.41340885848751E-17" rpy="0 0 0" />
-      <mass value="0.00231470671016277" />
+      <mass value="${roller_mass}" />
       <inertia
       ixx="8.41931982734933E-08" ixy="2.06795153138257E-25" ixz="1.77456090786767E-23"
@@ -87,5 +91,5 @@
     <inertial>
       <origin xyz="0 0 8.5868812060852E-17" rpy="0 0 0" />
-      <mass value="0.00231470671016277" />
+      <mass value="${roller_mass}" />
       <inertia
       ixx="8.41931982734976E-08" ixy="-7.10858338912758E-26" ixz="1.15805285757424E-23"
@@ -115,5 +119,5 @@
     <inertial>
       <origin xyz="6.93889390390723E-18 -1.38777878078145E-17 8.32667268468867E-17" rpy="0 0 0" />
-      <mass value="0.00231470671016277" />
+      <mass value="${roller_mass}" />
       <inertia
       ixx="8.4193198273496E-08" ixy="1.24077091882954E-24" ixz="-6.61744490042422E-24"
@@ -143,5 +147,5 @@
     <inertial>
       <origin xyz="0 -2.77555756156289E-17 8.5868812060852E-17" rpy="0 0 0" />
-      <mass value="0.00231470671016277" />
+      <mass value="${roller_mass}" />
       <inertia
       ixx="8.41931982734932E-08" ixy="4.13590306276514E-25" ixz="2.31610571514848E-23"
@@ -171,5 +175,5 @@
     <inertial>
       <origin xyz="0 0 8.67361737988404E-17" rpy="0 0 0" />
-      <mass value="0.00231470671016277" />
+      <mass value="${roller_mass}" />
       <inertia
       ixx="8.41931982734933E-08" ixy="-2.66652656448979E-24" ixz="1.39586728368323E-23"
@@ -199,5 +203,5 @@
     <inertial>
       <origin xyz="5.20417042793042E-18 0 8.8037216405823E-17" rpy="0 0 0" />
-      <mass value="0.00231470671016277" />
+      <mass value="${roller_mass}" />
       <inertia
       ixx="8.41931982734933E-08" ixy="8.27180612553028E-25" ixz="1.57164316385075E-23"
@@ -227,5 +231,5 @@
     <inertial>
       <origin xyz="6.93889390390723E-18 0 7.80625564189563E-17" rpy="0 0 0" />
-      <mass value="0.00231470671016277" />
+      <mass value="${roller_mass}" />
       <inertia
       ixx="8.41931982734933E-08" ixy="4.87907314435575E-25" ixz="1.31314922242793E-23"
@@ -255,5 +259,5 @@
     <inertial>
       <origin xyz="6.93889390390723E-18 0 -8.50014503228635E-17" rpy="0 0 0" />
-      <mass value="0.00231470671016277" />
+      <mass value="${roller_mass}" />
       <inertia
       ixx="8.41931982734933E-08" ixy="-1.65436122510606E-24" ixz="5.16987882845642E-24"
@@ -283,5 +287,5 @@
     <inertial>
       <origin xyz="0 0 8.84708972748172E-17" rpy="0 0 0" />
-      <mass value="0.00231470671016277" />
+      <mass value="${roller_mass}" />
       <inertia
       ixx="8.41931982734928E-08" ixy="-4.13590306276514E-25" ixz="1.81979734761666E-23"
@@ -311,5 +315,5 @@
     <inertial>
       <origin xyz="0 -1.38777878078145E-17 8.67361737988404E-17" rpy="0 0 0" />
-      <mass value="0.00231470671016277" />
+      <mass value="${roller_mass}" />
       <inertia
       ixx="8.41931982734964E-08" ixy="-1.24077091882954E-24" ixz="1.65436122510606E-24"
@@ -339,5 +343,5 @@
     <inertial>
       <origin xyz="8.27907396198134E-05 2.56280149801419E-05 6.93889390390723E-18" rpy="0 0 0" />
-      <mass value="0.0479080577376475" />
+      <mass value="${hub_mass}" />
       <inertia
       ixx="6.92600027574926E-06" ixy="2.68210543382497E-08" ixz="-5.90487790310826E-10"
@@ -367,5 +371,5 @@
     <inertial>
       <origin xyz="-4.38538094726937E-15 2.8943861196673E-14 -1.66533453693773E-16" rpy="0 0 0" />
-      <mass value="0.00231470671016277" />
+      <mass value="${roller_mass}" />
       <inertia
       ixx="8.41931982734932E-08" ixy="8.16840854896115E-24" ixz="1.88054342385102E-23"
@@ -395,5 +399,5 @@
     <inertial>
       <origin xyz="5.70377078901174E-15 -8.02136135291676E-15 2.50381312905112E-14" rpy="0 0 0" />
-      <mass value="0.00231470671016277" />
+      <mass value="${roller_mass}" />
       <inertia
       ixx="8.41931982734928E-08" ixy="1.32348898008484E-23" ixz="2.56425989891439E-23"
@@ -423,5 +427,5 @@
     <inertial>
       <origin xyz="2.08895400977127E-14 7.84095011141517E-15 1.64191577001205E-14" rpy="0 0 0" />
-      <mass value="0.00231470671016277" />
+      <mass value="${roller_mass}" />
       <inertia
       ixx="8.41931982734978E-08" ixy="-2.48154183765908E-24" ixz="2.48154183765908E-23"
@@ -451,5 +455,5 @@
     <inertial>
       <origin xyz="1.74721348500384E-14 -1.60912949631609E-14 -1.50695428358105E-14" rpy="0 0 0" />
-      <mass value="0.00231470671016277" />
+      <mass value="${roller_mass}" />
       <inertia
       ixx="8.41931982734926E-08" ixy="-4.13590306276514E-24" ixz="2.8951321439356E-23"
@@ -479,5 +483,5 @@
     <inertial>
       <origin xyz="-4.02455846426619E-16 -8.12544476147536E-15 -2.53234933023094E-14" rpy="0 0 0" />
-      <mass value="0.00231470671016277" />
+      <mass value="${roller_mass}" />
       <inertia
       ixx="8.41931982734987E-08" ixy="2.06795153138257E-25" ixz="9.15068552636787E-24"
@@ -507,5 +511,5 @@
     <inertial>
       <origin xyz="-7.82707232360735E-15 2.23467078175332E-14 1.49914802793916E-14" rpy="0 0 0" />
-      <mass value="0.00231470671016277" />
+      <mass value="${roller_mass}" />
       <inertia
       ixx="8.41931982734932E-08" ixy="-8.27180612553028E-25" ixz="1.3648480107125E-23"
@@ -535,5 +539,5 @@
     <inertial>
       <origin xyz="1.38777878078145E-17 -3.46944695195361E-18 7.97972798949331E-17" rpy="0 0 0" />
-      <mass value="0.00231470671016277" />
+      <mass value="${roller_mass}" />
       <inertia
         ixx="8.41931982734977E-08" ixy="2.06795153138257E-24" ixz="1.0998917207541E-23"
@@ -563,5 +567,5 @@
     <inertial>
       <origin xyz="0 -6.93889390390723E-18 8.50014503228635E-17" rpy="0 0 0" />
-      <mass value="0.00231470671016277" />
+      <mass value="${roller_mass}" />
       <inertia
       ixx="8.41931982734932E-08" ixy="-6.51751831183807E-24" ixz="1.24691014993833E-23"
@@ -591,5 +595,5 @@
     <inertial>
       <origin xyz="-3.46944695195361E-18 6.93889390390723E-18 8.32667268468867E-17" rpy="0 0 0" />
-      <mass value="0.00231470671016277" />
+      <mass value="${roller_mass}" />
       <inertia
       ixx="8.41931982734977E-08" ixy="3.30872245021211E-24" ixz="1.81979734761666E-23"
@@ -619,5 +623,5 @@
     <inertial>
       <origin xyz="-3.46944695195361E-18 6.93889390390723E-18 8.50014503228635E-17" rpy="0 0 0" />
-      <mass value="0.00231470671016277" />
+      <mass value="${roller_mass}" />
       <inertia
       ixx="8.41931982734963E-08" ixy="8.27180612553028E-25" ixz="1.15805285757424E-23"
@@ -647,5 +651,5 @@
     <inertial>
       <origin xyz="2.56280149801454E-05 -8.27907396198091E-05 0" rpy="0 0 0" />
-      <mass value="0.0479080577376475" />
+      <mass value="${hub_mass}" />
       <inertia
       ixx="6.84765795190243E-06" ixy="-2.68210543382476E-08" ixz="1.90755783989289E-09"
@@ -675,5 +679,5 @@
     <inertial>
       <origin xyz="-1.38777878078145E-16 6.31439345255558E-16 1.57859836313889E-16" rpy="0 0 0" />
-      <mass value="0.00231470671016277" />
+      <mass value="${roller_mass}" />
       <inertia
       ixx="8.41931982734932E-08" ixy="-8.96973976737189E-24" ixz="1.55096364853693E-23"
@@ -703,5 +707,5 @@
     <inertial>
       <origin xyz="5.45397060847108E-15 -3.49026363366534E-15 3.17714604625152E-14" rpy="0 0 0" />
-      <mass value="0.00231470671016278" />
+      <mass value="${roller_mass}" />
       <inertia
       ixx="8.41931982734995E-08" ixy="-6.61744490042422E-24" ixz="2.48154183765908E-24"
@@ -731,5 +735,5 @@
     <inertial>
       <origin xyz="6.93889390390723E-18 -1.38777878078145E-17 8.67361737988404E-17" rpy="0 0 0" />
-      <mass value="0.00231470671016277" />
+      <mass value="${roller_mass}" />
       <inertia
       ixx="8.41931982734975E-08" ixy="1.02363600803437E-23" ixz="1.65436122510606E-23"
@@ -759,5 +763,5 @@
     <inertial>
       <origin xyz="-2.08166817117217E-17 6.93889390390723E-18 9.0205620750794E-17" rpy="0 0 0" />
-      <mass value="0.00231470671016277" />
+      <mass value="${roller_mass}" />
       <inertia
       ixx="8.41931982734893E-08" ixy="4.96308367531817E-24" ixz="1.32348898008484E-23"
@@ -787,5 +791,5 @@
     <inertial>
       <origin xyz="6.09928774153445E-15 8.67361737988404E-16 -2.62116717220096E-14" rpy="0 0 0" />
-      <mass value="0.00231470671016277" />
+      <mass value="${roller_mass}" />
       <inertia
       ixx="8.4193198273491E-08" ixy="9.92616735063633E-24" ixz="3.14328632770151E-23"
@@ -815,5 +819,5 @@
     <inertial>
       <origin xyz="1.08593689596148E-14 3.19813620031084E-14 1.24067423001861E-14" rpy="0 0 0" />
-      <mass value="0.00231470671016277" />
+      <mass value="${roller_mass}" />
       <inertia
       ixx="8.41931982734964E-08" ixy="5.37667398159468E-24" ixz="-1.65436122510606E-24"
@@ -843,5 +847,5 @@
     <inertial>
       <origin xyz="1.83186799063151E-15 -2.58126853225349E-15 1.14248888127833E-14" rpy="0 0 0" />
-      <mass value="0.00231470671016277" />
+      <mass value="${roller_mass}" />
       <inertia
       ixx="8.41931982734904E-08" ixy="3.30872245021211E-24" ixz="1.03397576569128E-23"
@@ -871,5 +875,5 @@
     <inertial>
       <origin xyz="1.35039548987415E-14 0 1.5560469579512E-15" rpy="0 0 0" />
-      <mass value="0.00231470671016277" />
+      <mass value="${roller_mass}" />
       <inertia
       ixx="8.41931982734933E-08" ixy="2.22304789623626E-24" ixz="1.69572025573371E-23"
@@ -899,5 +903,5 @@
     <inertial>
       <origin xyz="-1.38777878078145E-17 0 8.50014503228635E-17" rpy="0 0 0" />
-      <mass value="0.00231470671016277" />
+      <mass value="${roller_mass}" />
       <inertia
       ixx="8.41931982734934E-08" ixy="-6.61744490042422E-24" ixz="5.79026428787119E-24"
@@ -927,5 +931,5 @@
     <inertial>
       <origin xyz="0 -6.93889390390723E-18 8.32667268468867E-17" rpy="0 0 0" />
-      <mass value="0.00231470671016277" />
+      <mass value="${roller_mass}" />
       <inertia
       ixx="8.41931982734928E-08" ixy="-3.51551760335037E-24" ixz="1.65436122510606E-23"
